Commit message: 修改安川机器人呢urdf文件,包括: 1. 修改2,3轴的方向 2. 修改2轴的限位方向(文档中上下限位与实际不同)
添加ABB 1410机器人的角度替换宏定义,当不使用该宏时,不对第三轴角度进行修正

File: SpraySystem/Trajectory/Libs/urdf/mpx2600/urdf/mpx2600_urdf.urdf (robot description, URDF)
Before this commit: robot mpx2600_urdf, 9 links, 8 joints
Joints:
- joint joint2: axis 0 1 0 -> 0 -1 0; limit lower=-1.1345 upper=2.2689 effort=0 velocity=2.09 -> lower=-2.26892 upper=1.1344 effort=0 velocity=2.09
- joint joint3: axis 0 1 0 -> 0 -1 0; limit lower=-1.1345 upper=2.618 effort=0 velocity=2.18 -> lower=-1.0646 upper=2.6179 effort=0 velocity=2.18
- joint joint4: limit lower=-12.5664 upper=12.5664 effort=0 velocity=6.28 -> lower=-5.0000 upper=5.0000 effort=0 velocity=6.28
- joint joint5: limit lower=-12.5664 upper=12.5664 effort=0 velocity=6.28 -> lower=-5.0000 upper=5.0000 effort=0 velocity=6.28
- joint joint6: limit lower=-12.5664 upper=12.5664 effort=0 velocity=6.28 -> lower=-5.0000 upper=5.0000 effort=0 velocity=6.28
- joint joint_flange: origin xyz=0 0 0 rpy=0 1.57 0 -> xyz=0.1 0 0 rpy=0 1.57 0

Commit message: 修改规划模式, 在规划空间自由曲线时,添加一次非ompl规划,并且采用关节角插值的初始化

File: SpraySystem/Trajectory/Libs/urdf/mpx2600/urdf/mpx2600_urdf.urdf (robot description, URDF)
Before this commit: robot mpx2600_urdf, 9 links, 8 joints
Joints:
- joint joint3: limit lower=-1.0646 upper=2.6179 effort=0 velocity=2.18 -> lower=-1.08 upper=2.6179 effort=0 velocity=2.18
- joint joint4: limit lower=-5.0000 upper=5.0000 effort=0 velocity=6.28 -> lower=-6.28 upper=6.28 effort=0 velocity=6.28
- joint joint5: limit lower=-5.0000 upper=5.0000 effort=0 velocity=6.28 -> lower=-6.28 upper=6.28 effort=0 velocity=6.28
- joint joint6: limit lower=-5.0000 upper=5.0000 effort=0 velocity=6.28 -> lower=-6.28 upper=6.28 effort=0 velocity=6.28

Commit message: 修改了安川机器人的urdf，取消了yaskawa_offset的宏定义 添加了地轨和阻挡

File: SpraySystem/Trajectory/Libs/urdf/mpx2600/urdf/mpx2600_urdf.urdf (robot description, URDF)
Before this commit: robot mpx2600_urdf, 9 links, 8 joints
Joints:
- joint joint1: origin xyz=-0.15844 0 0.2515 rpy=0 0 0 -> xyz=0 0 -0.3485 rpy=0 0 0
- joint joint4: limit lower=-6.28 upper=6.28 effort=0 velocity=6.28 -> lower=-6.283185307 upper=6.283185307 effort=0 velocity=6.283185307
- joint joint5: limit lower=-6.28 upper=6.28 effort=0 velocity=6.28 -> lower=-6.283185307 upper=6.283185307 effort=0 velocity=6.283185307
- joint joint6: limit lower=-6.28 upper=6.28 effort=0 velocity=6.28 -> lower=-6.283185307 upper=6.283185307 effort=0 velocity=6.283185307

Commit message: 1. 视觉添加新新方法区分计算头部和尾部中心点；

File: SpraySystem/Trajectory/Libs/urdf/mpx2600/urdf/mpx2600_urdf.urdf (robot description, URDF)
Before this commit: robot mpx2600_urdf, 9 links, 8 joints
Links:
- link link_painter: geometry collision box size=0.85 0.1 0.75; visual box size=0.85 0.1 0.75
Joints:
- joint joint4: limit lower=-6.283185307 upper=6.283185307 effort=0 velocity=6.283185307 -> lower=-12.56636 upper=12.56636 effort=0 velocity=6.283185307
- joint joint5: limit lower=-6.283185307 upper=6.283185307 effort=0 velocity=6.283185307 -> lower=-12.56636 upper=12.56636 effort=0 velocity=6.283185307
- joint joint6: limit lower=-6.283185307 upper=6.283185307 effort=0 velocity=6.283185307 -> lower=-12.56636 upper=12.56636 effort=0 velocity=6.283185307

Commit message: 1. 添加悬挂链,调整了场景参数, 2. 添加了安全目的障碍物

File: SpraySystem/Trajectory/Libs/urdf/mpx2600/urdf/mpx2600_urdf.urdf (robot description, URDF)
Before this commit: robot mpx2600_urdf, 9 links, 8 joints
Links:
- link link_painter: geometry collision box size=0.7 0.1 0.6; visual box size=0.7 0.1 0.6
